File: v1.0/hardware/eous-v1.0.kicad_sch (KiCad schematic)
At the start: 67 parts, among them J1 Screw_Terminal_01x02, U1 BQ25883RGER, U2 ICM-45686, U3 STM32F722RETx, U4 BMP580, U5 TPS63070RNMR, U6 LMR51430

Commit message: layout pcb
Parts:
- removed FB1: FerriteBead_Small, symbol Device:FerriteBead_Small
- added C33, C34: 20pF, Capacitor_SMD:C_0201_0603Metric, symbol Device:C_Small
- added C35, C36: 6.8pF, Capacitor_SMD:C_0201_0603Metric, symbol Device:C_Small
- added C37: 100nF, Capacitor_SMD:C_0201_0603Metric, symbol Device:C_Small
- added J2, J3: Conn_01x03, Connector_PinHeader_2.54mm:PinHeader_1x03_P2.54mm_Vertical, symbol Connector_Generic:Conn_01x03
- added L4: FCM1608KF-601T03, lcsc:L0603, symbol lcsc:FCM1608KF-601T03
- added R22: 10K, Resistor_SMD:R_0201_0603Metric, symbol Device:R_Small
- added SW1, SW2: TS-1088-AR02016, lcsc:SW-SMD_L3.9-W3.0-P4.45, symbol lcsc:TS-1088-AR02016
- added X1: X322525MOB4SI, lcsc:CRYSTAL-SMD_4P-L3.2-W2.5-BL, symbol lcsc:X322525MOB4SI
- added X2: Q13FC1350000400, lcsc:FC-135R_L3.2-W1.5, symbol lcsc:Q13FC1350000400
- C1: value 10uF -> 1uF; footprint (none) -> Capacitor_SMD:C_0402_1005Metric
- C10, C12, C13, C14, C9: footprint (none) -> Capacitor_SMD:C_0805_2012Metric
- C11, C17, C8: footprint (none) -> Capacitor_SMD:C_0603_1608Metric
- C15, C19, C20, C21, C22, C23, C24, C25, C26, C27, C28, C3, C7: footprint (none) -> Capacitor_SMD:C_0201_0603Metric
- C16, C18, C2, C29, C30, C31, C32, C6: footprint (none) -> Capacitor_SMD:C_0402_1005Metric
- C4: value 47nF -> 10uF; footprint (none) -> Capacitor_SMD:C_0603_1608Metric
- C5: value 10uF -> 44uF; footprint (none) -> Capacitor_SMD:C_0603_1608Metric
- Card1: footprint easyeda2kicad:TF-SMD_TF-01A -> lcsc:TF-SMD_TF-01A
- D1: footprint (none) -> LED_SMD:LED_0402_1005Metric
- J1: footprint (none) -> TerminalBlock:TerminalBlock_Xinya_XY308-2.54-2P_1x02_P2.54mm_Horizontal
- L1: footprint (none) -> lcsc:L2520
- L2: footprint (none) -> lcsc:IND-SMD_L4.0-W4.0-A
- L3: footprint (none) -> lcsc:IND-SMD_L3.0-W3.0
- R1, R10, R11, R12, R16, R17, R18, R19, R2, R20, R21, R3, R4, R5, R6, R7, R8, R9: footprint (none) -> Resistor_SMD:R_0201_0603Metric
- R13, R14, R15: footprint (none) -> Resistor_SMD:R_0402_1005Metric
- U1: footprint easyeda2kicad:VFQFPN-24_L4.0-W4.0-P0.50-BL-EP2.8 -> lcsc:VFQFPN-24_L4.0-W4.0-P0.50-BL-EP2.8
- U2: footprint easyeda2kicad:LGA-14_L3.0-W2.5-P0.50-TL -> lcsc:LGA-14_L3.0-W2.5-P0.50-TL
- U4: footprint easyeda2kicad:LGA-10_L2.0-W2.0-P0.50-TL_BMP580 -> lcsc:LGA-10_L2.0-W2.0-P0.50-TL_BMP580
- U5: footprint easyeda2kicad:VQFN-15_L3.0-W2.5-P0.50-BL -> lcsc:VQFN-15_L3.0-W2.5-P0.50-BL
- USB1: footprint easyeda2kicad:USB-C-SMD_TYPE-C-16PIN-2MD-073 -> lcsc:USB-C-SMD_TYPE-C-16PIN-2MD-073
Connections:
- net +3.3V: now also L4.2, SW2.1
- net +5V: now also J2.1 (Pin_1), J3.1 (Pin_1)
- net BMP_INT: now also U3.62 (PB9)
- net BQ_CE: now also U3.61 (PB8)
- net BQ_INT: now also U3.57 (PB5)
- net GND: now also C33.2, C34.2, C35.2, C36.2, C37.1, J2.3 (Pin_3), J3.3 (Pin_3), R22.2, SW1.1, X1.2 (GND), X1.4 (GND)
- net I2C_SCL: now also U3.58 (PB6)
- net I2C_SDA: now also U3.59 (PB7)
- net ICM_CS: now also U3.20 (PA4)
- net ICM_INT1: now also U3.24 (PC4)
- net ICM_INT2: now also U3.25 (PB0)
- net ICM_SCK: now also U3.21 (PA5)
- net ICM_SDI: now also U3.23 (PA7)
- net ICM_SDO: now also U3.22 (PA6)
- net SD_CD: now also U3.55 (PB3)
- net SD_CLK: now also U3.53 (PC12)
- net SD_CMD: now also U3.54 (PD2)
- net SD_DAT0: now also U3.39 (PC8)
- net SD_DAT1: now also U3.40 (PC9)
- net SD_DAT2: now also U3.51 (PC10)
- net SD_DAT3: now also U3.52 (PC11)
- net USB_DN: now also U3.44 (PA11)
- net USB_DP: now also U3.45 (PA12)
- net at U3.13 (VDDA): now also L4.1
- net SERVO1: now reaches U3.14 (PA0)
- net SERVO1: now also J2.2 (Pin_2)
- net SERVO2: now reaches U3.15 (PA1)
- net SERVO2: now also J3.2 (Pin_2)
- net LSE_IN: now reaches U3.3 (PC14)
- net LSE_IN: now also C35.1, X2.1
- net LSE_OUT: now reaches U3.4 (PC15)
- net LSE_OUT: now also C36.1, X2.2
- net HSE_IN: now reaches U3.5 (PH0)
- net HSE_IN: now also C33.1, X1.1 (OSC1)
- net HSE_OUT: now reaches U3.6 (PH1)
- net HSE_OUT: now also C34.1, X1.3 (OSC2)
- net BOOT: now reaches U3.60 (BOOT0)
- net BOOT: now also R22.1, SW2.2
- net RESET: now reaches U3.7 (NRST)
- net RESET: now also C37.2, SW1.2
- no-connect marks 10 -> 34
Other:
- note added: "3.3V buck"
- note added: "5V buck-boost"
- note added: "BOOT/RESET Buttons"
- note added: "Barometer"
- note added: "Battery Charger IC"
- note added: "Clock"
- note added: "Eous"
- note added: "IMU"
- note added: "Power decoupling"
- note added: "SD Card"
- note added: "STM32"
- note added: "TVC Servos"
- note added: "USB-C Port"
- title: Eous -> TVC Flight Controller
- moved on the sheet: C10, C11, C12, C13, C14, C15, C16, C17, C18, C19, C20, C21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
